File: power.kicad_sch (KiCad schematic)
At the start: 21 parts, among them U401 LM66200DRLR, U402 MAX77827AEFD+T, U403 SC4215

Commit message: File names and ERC
Parts:
- renumbered C401 to C20, C402 to C21, C404 to C22, C405 to C23, C406 to C24, C407 to C25, C408 to C26, C403 to C27, L401 to L3, R401 to R14, R403 to R15, R404 to R16, R402 to R17, TP401 to TP10, TP402 to TP6, TP403 to TP7, TP404 to TP8, TP405 to TP9, U401 to U3, U403 to U4, U402 to U5

Commit message: Add photo triggers
Parts:
- U3: footprint iclr:SOTFL50P160X60-8N -> fps:SOTFL50P160X60-8N
- U4: footprint iclr:SOIC127P599X175-9N -> fps:SOIC127P599X175-8N
- U5: footprint iclr:CONV_MAX77827AEFD+T -> fps:CONV_MAX77827AEFD+T
Changed lines of the file:
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@@
       (effects (font (size 1.27 1.27)))
     )
-    (property "Footprint" "iclr:SOTFL50P160X60-8N" (at 76.2 34.29 0)
+    (property "Footprint" "fps:SOTFL50P160X60-8N" (at 76.2 34.29 0)
       (effects (font (size 1.27 1.27)) (justify left) hide)
     )
@@
       (effects (font (size 1.27 1.27)))
     )
-    (property "Footprint" "iclr:SOIC127P599X175-9N" (at 218.44 45.72 0)
+    (property "Footprint" "fps:SOIC127P599X175-8N" (at 218.44 45.72 0)
       (effects (font (size 1.27 1.27)) hide)
     )
@@
       (effects (font (size 1.27 1.27)))
     )
-    (property "Footprint" "iclr:CONV_MAX77827AEFD+T" (at 144.78 43.18 0)
+    (property "Footprint" "fps:CONV_MAX77827AEFD+T" (at 144.78 43.18 0)
       (effects (font (size 1.27 1.27)) (justify left bottom) hide)
     )

Commit message: Fixed libraries and footprints
Connections:
- net GND: no longer U4.9 (GND)
- no-connect marks 4 -> 5
Changed lines of the file:
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@@
   (junction (at 200.66 52.07) (diameter 0) (color 0 0 0 0)
   )
+  (no_connect (at 215.9 67.31))
   (no_connect (at 166.37 67.31))
   (no_connect (at 135.89 59.69))
@@
   )
   (wire (pts (xy 240.03 60.96) (xy 240.03 62.23))
+    (stroke (width 0) (type default))
+  )
+  (wire (pts (xy 218.44 67.31) (xy 218.44 69.85))
     (stroke (width 0) (type default))
   )
@@
     )
   )
-  (symbol (lib_id "power:GND") (at 218.44 67.31 0) (unit 1)
-    (in_bom yes) (on_board yes) (dnp no)
-    (property "Reference" "#PWR047" (at 218.44 73.66 0)
-      (effects (font (size 1.27 1.27)) hide)
-    )
-    (property "Value" "GND" (at 218.44 71.12 0)
-      (effects (font (size 1.27 1.27)))
-    )
-    (property "Footprint" "" (at 218.44 67.31 0)
-      (effects (font (size 1.27 1.27)) hide)
-    )
-    (property "Datasheet" "" (at 218.44 67.31 0)
+  (symbol (lib_id "power:GND") (at 218.44 69.85 0) (unit 1)
+    (in_bom yes) (on_board yes) (dnp no)
+    (property "Reference" "#PWR047" (at 218.44 76.2 0)
+      (effects (font (size 1.27 1.27)) hide)
+    )
+    (property "Value" "GND" (at 218.44 73.66 0)
+      (effects (font (size 1.27 1.27)))
+    )
+    (property "Footprint" "" (at 218.44 69.85 0)
+      (effects (font (size 1.27 1.27)) hide)
+    )
+    (property "Datasheet" "" (at 218.44 69.85 0)
       (effects (font (size 1.27 1.27)) hide)
     )
@@
     (pin "3")
     (pin "4")
+    (pin "5")
     (pin "6")
     (pin "7")
     (pin "8")
-    (pin "9")
-    (instances
-      (project "RicardoCHEESE"
+    (instances
+      (project "RicardoCHEESE"

Commit message: Footprinting and board outline
Parts:
- C23, C24: footprint Capacitor_SMD:C_0603_1608Metric -> Capacitor_SMD:C_0402_1005Metric
Changed lines of the file:
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@@
       (effects (font (size 1.27 1.27)) (justify left))
     )
-    (property "Footprint" "Capacitor_SMD:C_0603_1608Metric" (at 184.15 54.61 0)
+    (property "Footprint" "Capacitor_SMD:C_0402_1005Metric" (at 184.15 54.61 0)
       (effects (font (size 1.27 1.27)) hide)
     )
@@
       (effects (font (size 1.27 1.27)) (justify left))
     )
-    (property "Footprint" "Capacitor_SMD:C_0603_1608Metric" (at 194.31 54.61 0)
-      (effects (font (size 1.27 1.27)) hide)
-    )
+    (property "Footprint" "Capacitor_SMD:C_0402_1005Metric" (at 194.31 54.61 0)
+      (effects (font (size 1.27 1.27)) hide)
+    )

Commit message: radio side needs reviewing
Parts:
- C22: footprint Capacitor_SMD:C_0805_2012Metric -> Capacitor_SMD:C_0603_1608Metric
- C27: footprint Capacitor_SMD:C_0603_1608Metric -> Capacitor_SMD:C_0402_1005Metric
- U3: footprint fps:SOTFL50P160X60-8N -> iclr:SOTFL50P160X60-8N
- U4: footprint fps:SOIC127P599X175-8N -> iclr:SOIC127P599X175-8N
- U5: footprint fps:CONV_MAX77827AEFD+T -> iclr:CONV_MAX77827AEFD+T
Connections:
- net VoutDiode is gone; now on net BBIN: U3.2 (VOUT_1), U3.7 (VOUT_2)
Changed lines of the file:
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@@
+    (effects (font (size 1.27 1.27)) (justify right bottom))
+  )
+  (label "VoutDiode" (at 101.6 52.07 180) (fields_autoplaced)
     (effects (font (size 1.27 1.27)) (justify right bottom))
   )
@@
       (effects (font (size 1.27 1.27)))
     )
-    (property "Footprint" "fps:SOTFL50P160X60-8N" (at 76.2 34.29 0)
+    (property "Footprint" "iclr:SOTFL50P160X60-8N" (at 76.2 34.29 0)
       (effects (font (size 1.27 1.27)) (justify left) hide)
     )
@@
       (effects (font (size 1.27 1.27)))
     )
-    (property "Footprint" "fps:SOIC127P599X175-8N" (at 218.44 45.72 0)
+    (property "Footprint" "iclr:SOIC127P599X175-8N" (at 218.44 45.72 0)
       (effects (font (size 1.27 1.27)) hide)
     )
@@
       (effects (font (size 1.27 1.27)))
     )
-    (property "Footprint" "fps:CONV_MAX77827AEFD+T" (at 144.78 43.18 0)
+    (property "Footprint" "iclr:CONV_MAX77827AEFD+T" (at 144.78 43.18 0)
       (effects (font (size 1.27 1.27)) (justify left bottom) hide)
     )
@@
       (effects (font (size 1.27 1.27)) (justify left))
     )
-    (property "Footprint" "Capacitor_SMD:C_0805_2012Metric" (at 179.07 54.61 0)
+    (property "Footprint" "Capacitor_SMD:C_0603_1608Metric" (at 179.07 54.61 0)
       (effects (font (size 1.27 1.27)) hide)
     )
@@
       (effects (font (size 1.27 1.27)) (justify left))
     )
-    (property "Footprint" "Capacitor_SMD:C_0603_1608Metric" (at 132.08 69.85 0)
-      (effects (font (size 1.27 1.27)) hide)
-    )
+    (property "Footprint" "Capacitor_SMD:C_0402_1005Metric" (at 132.08 69.85 0)
+      (effects (font (size 1.27 1.27)) hide)
+    )

Commit message: post andrei review
Parts:
- C25: footprint Capacitor_SMD:C_0603_1608Metric -> Capacitor_SMD:C_0402_1005Metric
- U4: footprint iclr:SOIC127P599X175-8N -> iclr:SOIC127P599X175-9N
Changed lines of the file:
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@@
       (effects (font (size 1.27 1.27)) (justify right))
     )
-    (property "Footprint" "Capacitor_SMD:C_0603_1608Metric" (at 252.73 54.61 0)
+    (property "Footprint" "Capacitor_SMD:C_0402_1005Metric" (at 252.73 54.61 0)
       (effects (font (size 1.27 1.27)) hide)
     )
@@
       (effects (font (size 1.27 1.27)))
     )
-    (property "Footprint" "iclr:SOIC127P599X175-8N" (at 218.44 45.72 0)
+    (property "Footprint" "iclr:SOIC127P599X175-9N" (at 218.44 45.72 0)
       (effects (font (size 1.27 1.27)) hide)
     )
