File: power.kicad_sch (KiCad schematic)
At the start: 21 parts, among them U3 LM66200DRLR, U4 SC4215, U5 MAX77827AEFD+T

Commit message: ordering
Connections:
- net GND: now also U4.9 (GND)
Changed lines of the file:
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@@
     (pin "7")
     (pin "8")
+    (pin "9")
     (instances
       (project "RicardoCHEESE"
