File: camera.kicad_sch (KiCad schematic)
At the start: 42 parts, among them J3 Conn_Coaxial, J4 Conn_01x06_Pin, J5 Conn_01x06_Pin, J6 Conn_01x06_Pin, J7 Conn_01x06_Pin, U7 RTC6705, U8 HEF4051BT, Y2 8MHz

Commit message: post andrei review
Parts:
- C36, C42: value 33p -> 24p
- C37, C46: footprint Capacitor_SMD:C_0603_1608Metric -> Capacitor_SMD:C_0402_1005Metric
Connections:
- net +3.3V: now also U7.9 (V2D5_PLL)
- net +3.3VA: now also U7.40 (LDD2V5)
- net GND: now also Y2.2, Y2.4
- net at C36.1, Y2.1: now also U7.24 (XTAL1)
- net at C42.1, Y2.3: now also U7.25 (XTAL2)
- removed net OSC2: U7.24 (XTAL1), Y2.2
- removed net OSC4: U7.25 (XTAL2), Y2.4
- no-connect marks 18 -> 16
Other:
- moved on the sheet: Y2
