File: usb-uart.kicad_sch (KiCad schematic)
At the start: 9 parts, among them J10 USB_C_Receptacle_USB2.0

Commit message: File names and ERC
Parts:
- renumbered J10 to J2, R13 to R11, R11 to R12, R12 to R13, TP1 to TP3, TP2 to TP4, TP3 to TP5
Changed lines of the file:
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@@
   (symbol (lib_id "power:GND") (at 127 96.52 90) (unit 1)
     (in_bom yes) (on_board yes) (dnp no)
-    (property "Reference" "#PWR0121" (at 133.35 96.52 0)
+    (property "Reference" "#PWR032" (at 133.35 96.52 0)
       (effects (font (size 1.27 1.27)) hide)
     )
@@
     (pin "1")
     (instances
-      (project "RicardoCamera"
-        (path "/7db990e4-92e1-4f99-b4d2-435bbec1ba83/00000000-0000-0000-0000-000061925999"
-          (reference "#PWR0121") (unit 1)
+      (project "RicardoCHEESE"
+        (path "/7db990e4-92e1-4f99-b4d2-435bbec1ba83/00000000-0000-0000-0000-000061925999"
+          (reference "#PWR032") (unit 1)
         )
       )
@@
   (symbol (lib_id "Device:R_Small") (at 123.19 99.06 270) (unit 1)
     (in_bom yes) (on_board yes) (dnp no)
-    (property "Reference" "R12" (at 129.54 100.33 90)
+    (property "Reference" "R13" (at 129.54 100.33 90)
       (effects (font (size 1.27 1.27)))
     )
@@
     (pin "2")
     (instances
-      (project "RicardoCamera"
+      (project "RicardoCHEESE"
+        (path "/7db990e4-92e1-4f99-b4d2-435bbec1ba83/00000000-0000-0000-0000-000061925999"
+          (reference "R13") (unit 1)
+        )
+      )
+    )
+  )
+  (symbol (lib_id "Device:R_Small") (at 123.19 93.98 90) (unit 1)
+    (in_bom yes) (on_board yes) (dnp no)
+    (property "Reference" "R12" (at 123.19 89.0016 90)
+      (effects (font (size 1.27 1.27)))
+    )
+    (property "Value" "5.1k" (at 123.19 91.313 90)
+      (effects (font (size 1.27 1.27)))
+    )
+    (property "Footprint" "Resistor_SMD:R_0402_1005Metric" (at 123.19 93.98 0)
+      (effects (font (size 1.27 1.27)) hide)
+    )
+    (property "Datasheet" "~" (at 123.19 93.98 0)
+      (effects (font (size 1.27 1.27)) hide)
+    )
+    (pin "1")
+    (pin "2")
+    (instances
+      (project "RicardoCHEESE"
         (path "/7db990e4-92e1-4f99-b4d2-435bbec1ba83/00000000-0000-0000-0000-000061925999"
           (reference "R12") (unit 1)
@@
     )
   )
-  (symbol (lib_id "Device:R_Small") (at 123.19 93.98 90) (unit 1)
-    (in_bom yes) (on_board yes) (dnp no)
-    (property "Reference" "R11" (at 123.19 89.0016 90)
-      (effects (font (size 1.27 1.27)))
-    )
-    (property "Value" "5.1k" (at 123.19 91.313 90)
-      (effects (font (size 1.27 1.27)))
-    )
-    (property "Footprint" "Resistor_SMD:R_0402_1005Metric" (at 123.19 93.98 0)
-      (effects (font (size 1.27 1.27)) hide)
-    )
-    (property "Datasheet" "~" (at 123.19 93.98 0)
-      (effects (font (size 1.27 1.27)) hide)
-    )
-    (pin "1")
-    (pin "2")
-    (instances
-      (project "RicardoCamera"
-        (path "/7db990e4-92e1-4f99-b4d2-435bbec1ba83/00000000-0000-0000-0000-000061925999"
-          (reference "R11") (unit 1)
-        )
-      )
-    )
-  )
   (symbol (lib_id "power:GND") (at 96.52 130.81 0) (unit 1)
     (in_bom yes) (on_board yes) (dnp no)
-    (property "Reference" "#PWR0125" (at 96.52 137.16 0)
+    (property "Reference" "#PWR033" (at 96.52 137.16 0)
       (effects (font (size 1.27 1.27)) hide)
     )
@@
     (pin "1")
     (instances
-      (project "RicardoCamera"
-        (path "/7db990e4-92e1-4f99-b4d2-435bbec1ba83/00000000-0000-0000-0000-000061925999"
-          (reference "#PWR0125") (unit 1)
+      (project "RicardoCHEESE"
+        (path "/7db990e4-92e1-4f99-b4d2-435bbec1ba83/00000000-0000-0000-0000-000061925999"
+          (reference "#PWR033") (unit 1)
         )
       )
@@
   (symbol (lib_id "Connector:USB_C_Receptacle_USB2.0") (at 100.33 104.14 0) (unit 1)
     (in_bom yes) (on_board yes) (dnp no)
-    (property "Reference" "J10" (at 103.0478 82.1182 0)
+    (property "Reference" "J2" (at 103.0478 82.1182 0)
       (effects (font (size 1.27 1.27)))
     )
@@
     (pin "S1")
     (instances
-      (project "RicardoCamera"
-        (path "/7db990e4-92e1-4f99-b4d2-435bbec1ba83/00000000-0000-0000-0000-000061925999"
-          (reference "J10") (unit 1)
+      (project "RicardoCHEESE"
+        (path "/7db990e4-92e1-4f99-b4d2-435bbec1ba83/00000000-0000-0000-0000-000061925999"
+          (reference "J2") (unit 1)
         )
       )
@@
   (symbol (lib_id "power:GND") (at 132.08 144.78 0) (unit 1)
     (in_bom yes) (on_board yes) (dnp no)
-    (property "Reference" "#PWR0124" (at 132.08 151.13 0)
+    (property "Reference" "#PWR034" (at 132.08 151.13 0)
       (effects (font (size 1.27 1.27)) hide)
     )
@@
     (pin "1")
     (instances
-      (project "RicardoCamera"
-        (path "/7db990e4-92e1-4f99-b4d2-435bbec1ba83/00000000-0000-0000-0000-000061925999"
-          (reference "#PWR0124") (unit 1)
+      (project "RicardoCHEESE"
+        (path "/7db990e4-92e1-4f99-b4d2-435bbec1ba83/00000000-0000-0000-0000-000061925999"
+          (reference "#PWR034") (unit 1)
         )
       )
@@
     (pin "4")
     (instances
-      (project "RicardoCamera"
+      (project "RicardoCHEESE"
         (path "/7db990e4-92e1-4f99-b4d2-435bbec1ba83/00000000-0000-0000-0000-000061925999"
           (reference "D2") (unit 1)
@@
   (symbol (lib_id "power:VBUS") (at 116.84 85.09 0) (unit 1)
     (in_bom yes) (on_board yes) (dnp no)
-    (property "Reference" "#PWR0175" (at 116.84 88.9 0)
+    (property "Reference" "#PWR029" (at 116.84 88.9 0)
       (effects (font (size 1.27 1.27)) hide)
     )
@@
     (pin "1")
     (instances
-      (project "RicardoCamera"
-        (path "/7db990e4-92e1-4f99-b4d2-435bbec1ba83/00000000-0000-0000-0000-000061925999"
-          (reference "#PWR0175") (unit 1)
+      (project "RicardoCHEESE"
+        (path "/7db990e4-92e1-4f99-b4d2-435bbec1ba83/00000000-0000-0000-0000-000061925999"
+          (reference "#PWR029") (unit 1)
         )
       )
@@
   (symbol (lib_id "Connector:TestPoint") (at 52.07 99.06 270) (unit 1)
     (in_bom yes) (on_board yes) (dnp no)
-    (property "Reference" "TP1" (at 56.8452 97.8916 90)
+    (property "Reference" "TP3" (at 56.8452 97.8916 90)
       (effects (font (size 1.27 1.27)) (justify left))
     )
@@
     (pin "1")
     (instances
-      (project "RicardoCamera"
-        (path "/7db990e4-92e1-4f99-b4d2-435bbec1ba83/00000000-0000-0000-0000-000061925999"
-          (reference "TP1") (unit 1)
+      (project "RicardoCHEESE"
+        (path "/7db990e4-92e1-4f99-b4d2-435bbec1ba83/00000000-0000-0000-0000-000061925999"
+          (reference "TP3") (unit 1)
         )
       )
@@
   (symbol (lib_id "Connector:TestPoint") (at 52.07 104.14 270) (unit 1)
     (in_bom yes) (on_board yes) (dnp no)
-    (property "Reference" "TP2" (at 56.8452 102.9716 90)
+    (property "Reference" "TP4" (at 56.8452 102.9716 90)
       (effects (font (size 1.27 1.27)) (justify left))
     )
@@
     (pin "1")
     (instances
-      (project "RicardoCamera"
-        (path "/7db990e4-92e1-4f99-b4d2-435bbec1ba83/00000000-0000-0000-0000-000061925999"
-          (reference "TP2") (unit 1)
+      (project "RicardoCHEESE"
+        (path "/7db990e4-92e1-4f99-b4d2-435bbec1ba83/00000000-0000-0000-0000-000061925999"
+          (reference "TP4") (unit 1)
         )
       )
@@
   (symbol (lib_id "Connector:TestPoint") (at 52.07 109.22 270) (unit 1)
     (in_bom yes) (on_board yes) (dnp no)
-    (property "Reference" "TP3" (at 56.8452 108.0516 90)
+    (property "Reference" "TP5" (at 56.8452 108.0516 90)
       (effects (font (size 1.27 1.27)) (justify left))
     )
@@
     (pin "1")
     (instances
-      (project "RicardoCamera"
-        (path "/7db990e4-92e1-4f99-b4d2-435bbec1ba83/00000000-0000-0000-0000-000061925999"
-          (reference "TP3") (unit 1)
+      (project "RicardoCHEESE"
+        (path "/7db990e4-92e1-4f99-b4d2-435bbec1ba83/00000000-0000-0000-0000-000061925999"
+          (reference "TP5") (unit 1)
         )
       )
@@
     (pin "2")
     (instances
-      (project "RicardoCamera"
+      (project "RicardoCHEESE"
         (path "/7db990e4-92e1-4f99-b4d2-435bbec1ba83/00000000-0000-0000-0000-000061925999"
           (reference "USBLED1") (unit 1)
@@
   (symbol (lib_id "Device:R_Small") (at 154.94 92.71 90) (unit 1)
     (in_bom yes) (on_board yes) (dnp no)
-    (property "Reference" "R13" (at 154.94 97.6884 90)
+    (property "Reference" "R11" (at 154.94 97.6884 90)
       (effects (font (size 1.27 1.27)))
     )
@@
     (pin "2")
     (instances
-      (project "RicardoCamera"
-        (path "/7db990e4-92e1-4f99-b4d2-435bbec1ba83/00000000-0000-0000-0000-000061925999"
-          (reference "R13") (unit 1)
+      (project "RicardoCHEESE"
+        (path "/7db990e4-92e1-4f99-b4d2-435bbec1ba83/00000000-0000-0000-0000-000061925999"
+          (reference "R11") (unit 1)
         )
       )
@@
   (symbol (lib_id "power:GND") (at 165.1 92.71 90) (unit 1)
     (in_bom yes) (on_board yes) (dnp no)
-    (property "Reference" "#PWR0122" (at 171.45 92.71 0)
+    (property "Reference" "#PWR031" (at 171.45 92.71 0)
       (effects (font (size 1.27 1.27)) hide)
     )
@@
     (pin "1")
     (instances
-      (project "RicardoCamera"
-        (path "/7db990e4-92e1-4f99-b4d2-435bbec1ba83/00000000-0000-0000-0000-000061925999"
-          (reference "#PWR0122") (unit 1)
+      (project "RicardoCHEESE"
+        (path "/7db990e4-92e1-4f99-b4d2-435bbec1ba83/00000000-0000-0000-0000-000061925999"
+          (reference "#PWR031") (unit 1)
         )
       )
@@
   (symbol (lib_id "power:VBUS") (at 149.86 92.71 90) (unit 1)
     (in_bom yes) (on_board yes) (dnp no)
-    (property "Reference" "#PWR0174" (at 153.67 92.71 0)
+    (property "Reference" "#PWR030" (at 153.67 92.71 0)
       (effects (font (size 1.27 1.27)) hide)
     )
@@
     (pin "1")
     (instances
-      (project "RicardoCamera"
-        (path "/7db990e4-92e1-4f99-b4d2-435bbec1ba83/00000000-0000-0000-0000-000061925999"
-          (reference "#PWR0174") (unit 1)
-        )
-      )
+      (project "RicardoCHEESE"
+        (path "/7db990e4-92e1-4f99-b4d2-435bbec1ba83/00000000-0000-0000-0000-000061925999"
+          (reference "#PWR030") (unit 1)
+        )
+      )

Commit message: Camera buck changes, c and r footprints, other
Parts:
- J2: footprint Connector_USB:USB_C_Receptacle_GCT_USB4085 -> Connector_USB:USB_C_Receptacle_Palconn_UTC16-G
Changed lines of the file:
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@@
     (stroke (width 0) (type default))
   )
-  (wire (pts (xy 44.45 109.22) (xy 52.07 109.22))
+  (wire (pts (xy 31.75 109.22) (xy 52.07 109.22))
     (stroke (width 0) (type default))
   )
@@
   )
   (label "Data-" (at 116.84 102.87 0) (fields_autoplaced)
-    (effects (font (size 1.27 1.27)) (justify left bottom))
-  )
-  (label "VBUS" (at 44.45 109.22 0) (fields_autoplaced)
     (effects (font (size 1.27 1.27)) (justify left bottom))
   )
@@
     (effects (font (size 1.27 1.27)) (justify right))
   )
-  (hierarchical_label "VBUS" (shape input) (at 44.45 109.22 180) (fields_autoplaced)
-    (effects (font (size 1.27 1.27)) (justify right))
-  )
   (symbol (lib_id "power:GND") (at 127 96.52 90) (unit 1)
     (in_bom yes) (on_board yes) (dnp no)
@@
       (effects (font (size 1.27 1.27)))
     )
-    (property "Footprint" "Connector_USB:USB_C_Receptacle_GCT_USB4085" (at 104.14 104.14 0)
+    (property "Footprint" "Connector_USB:USB_C_Receptacle_Palconn_UTC16-G" (at 104.14 104.14 0)
       (effects (font (size 1.27 1.27)) hide)
     )
@@
         )
       )
+    )
+  )
+  (symbol (lib_id "power:VBUS") (at 31.75 109.22 0) (unit 1)
+    (in_bom yes) (on_board yes) (dnp no)
+    (property "Reference" "#PWR028" (at 31.75 113.03 0)
+      (effects (font (size 1.27 1.27)) hide)
+    )
+    (property "Value" "VBUS" (at 31.75 105.41 0)
+      (effects (font (size 1.27 1.27)))
+    )
+    (property "Footprint" "" (at 31.75 109.22 0)
+      (effects (font (size 1.27 1.27)) hide)
+    )
+    (property "Datasheet" "" (at 31.75 109.22 0)
+      (effects (font (size 1.27 1.27)) hide)
+    )
+    (pin "1")
+    (instances
+      (project "RicardoCHEESE"
+        (path "/7db990e4-92e1-4f99-b4d2-435bbec1ba83/00000000-0000-0000-0000-000061925999"
+          (reference "#PWR028") (unit 1)
+        )
+      )

Commit message: Finished routing
Connections:
- net Data+: now also D2.3 (K); no longer D2.4 (K)
- net Data-: now also D2.2 (K); no longer D2.3 (K)
- net VBUS: now also D2.4 (K); no longer D2.2 (K)
Changed lines of the file:
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@@
     (stroke (width 0) (type default))
   )
-  (label "Data+" (at 134.62 134.62 90) (fields_autoplaced)
+  (label "Data+" (at 132.08 134.62 90) (fields_autoplaced)
     (effects (font (size 1.27 1.27)) (justify left bottom))
   )
-  (label "VBUS" (at 129.54 134.62 90) (fields_autoplaced)
+  (label "VBUS" (at 134.62 134.62 90) (fields_autoplaced)
     (effects (font (size 1.27 1.27)) (justify left bottom))
   )
@@
     (effects (font (size 1.27 1.27)) (justify left bottom))
   )
-  (label "Data-" (at 132.08 134.62 90) (fields_autoplaced)
+  (label "Data-" (at 129.54 134.62 90) (fields_autoplaced)
     (effects (font (size 1.27 1.27)) (justify left bottom))
   )

Commit message: radio side needs reviewing
Parts:
- removed TP5: TestPoint, TestPoint:TestPoint_Pad_D1.0mm, symbol Connector:TestPoint
Changed lines of the file:
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@@
-    (stroke (width 0) (type default))
-  )
-  (wire (pts (xy 31.75 109.22) (xy 52.07 109.22))
     (stroke (width 0) (type default))
   )
@@
     )
     (property "Value" "TestPoint" (at 56.8452 105.283 90)
-      (effects (font (size 1.27 1.27)) (justify left))
+      (effects (font (size 1.27 1.27)) (justify left) hide)
     )
     (property "Footprint" "TestPoint:TestPoint_Pad_D1.0mm" (at 52.07 109.22 0)
@@
     )
   )
-  (symbol (lib_id "Connector:TestPoint") (at 52.07 109.22 270) (unit 1)
-    (in_bom yes) (on_board yes) (dnp no)
-    (property "Reference" "TP5" (at 56.8452 108.0516 90)
-      (effects (font (size 1.27 1.27)) (justify left))
-    )
-    (property "Value" "TestPoint" (at 56.8452 110.363 90)
-      (effects (font (size 1.27 1.27)) (justify left))
-    )
-    (property "Footprint" "TestPoint:TestPoint_Pad_D1.0mm" (at 52.07 114.3 0)
-      (effects (font (size 1.27 1.27)) hide)
-    )
-    (property "Datasheet" "~" (at 52.07 114.3 0)
-      (effects (font (size 1.27 1.27)) hide)
-    )
-    (pin "1")
-    (instances
-      (project "RicardoCHEESE"
-        (path "/7db990e4-92e1-4f99-b4d2-435bbec1ba83/00000000-0000-0000-0000-000061925999"
-          (reference "TP5") (unit 1)
-        )
-      )
-    )
-  )
   (symbol (lib_id "Device:LED_Small") (at 162.56 92.71 180) (unit 1)
     (in_bom yes) (on_board yes) (dnp no)
@@
         )
       )
-    )
-  )
-  (symbol (lib_id "power:VBUS") (at 31.75 109.22 0) (unit 1)
-    (in_bom yes) (on_board yes) (dnp no)
-    (property "Reference" "#PWR028" (at 31.75 113.03 0)
-      (effects (font (size 1.27 1.27)) hide)
-    )
-    (property "Value" "VBUS" (at 31.75 105.41 0)
-      (effects (font (size 1.27 1.27)))
-    )
-    (property "Footprint" "" (at 31.75 109.22 0)
-      (effects (font (size 1.27 1.27)) hide)
-    )
-    (property "Datasheet" "" (at 31.75 109.22 0)
-      (effects (font (size 1.27 1.27)) hide)
-    )
-    (pin "1")
-    (instances
-      (project "RicardoCHEESE"
-        (path "/7db990e4-92e1-4f99-b4d2-435bbec1ba83/00000000-0000-0000-0000-000061925999"
-          (reference "#PWR028") (unit 1)
-        )
-      )

Commit message: post andrei review
Parts:
- R11: value 470 -> 3000
Changed lines of the file:
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@@
       (effects (font (size 1.27 1.27)))
     )
-    (property "Value" "470" (at 154.94 95.377 90)
+    (property "Value" "3000" (at 154.94 95.377 90)
       (effects (font (size 1.27 1.27)))
     )
