File: RicardoCHEESE.kicad_sch (KiCad schematic)
At the start: 36 parts, among them J1 RBUS, U1 ESP32-S3, Y1 40MHz±10ppm

Commit message: post andrei review
Parts:
- removed 12VLED1: 12V_LED, LED_SMD:LED_0603_1608Metric, symbol Device:LED_Small
- removed R3: 3k, Resistor_SMD:R_0402_1005Metric, symbol Device:R_Small
Changed lines of the file:
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@@
   (junction (at 53.34 127) (diameter 0) (color 0 0 0 0)
-  )
-  (junction (at 58.42 26.67) (diameter 0) (color 0 0 0 0)
   )
   (junction (at 30.48 191.77) (diameter 0) (color 0 0 0 0)
@@
     (stroke (width 0) (type default))
   )
-  (wire (pts (xy 60.96 26.67) (xy 58.42 26.67))
-    (stroke (width 0) (type default))
-  )
   (wire (pts (xy 16.51 191.77) (xy 20.32 191.77))
     (stroke (width 0) (type default))
@@
     (stroke (width 0) (type default))
   )
-  (wire (pts (xy 58.42 21.59) (xy 58.42 26.67))
-    (stroke (width 0) (type default))
-  )
   (wire (pts (xy 161.29 138.43) (xy 156.21 138.43))
     (stroke (width 0) (type default))
@@
     (stroke (width 0) (type default))
   )
-  (wire (pts (xy 58.42 26.67) (xy 58.42 40.64))
+  (wire (pts (xy 58.42 21.59) (xy 58.42 40.64))
     (stroke (width 0) (type default))
   )
@@
   )
   (wire (pts (xy 53.34 127) (xy 55.88 127))
-    (stroke (width 0) (type default))
-  )
-  (wire (pts (xy 73.66 26.67) (xy 71.12 26.67))
     (stroke (width 0) (type default))
   )
@@
     )
   )
-  (symbol (lib_id "Device:LED_Small") (at 63.5 26.67 0) (unit 1)
-    (in_bom yes) (on_board yes) (dnp no)
-    (property "Reference" "12VLED1" (at 63.5 31.877 0)
-      (effects (font (size 1.27 1.27)))
-    )
-    (property "Value" "12V_LED" (at 63.5 29.5656 0)
-      (effects (font (size 1.27 1.27)))
-    )
-    (property "Footprint" "LED_SMD:LED_0603_1608Metric" (at 63.5 26.67 90)
-      (effects (font (size 1.27 1.27)) hide)
-    )
-    (property "Datasheet" "~" (at 63.5 26.67 90)
-      (effects (font (size 1.27 1.27)) hide)
-    )
-    (pin "1")
-    (pin "2")
-    (instances
-      (project "RicardoCHEESE"
-        (path "/7db990e4-92e1-4f99-b4d2-435bbec1ba83"
-          (reference "12VLED1") (unit 1)
-        )
-      )
-    )
-  )
-  (symbol (lib_id "Device:R_Small") (at 68.58 26.67 270) (unit 1)
-    (in_bom yes) (on_board yes) (dnp no)
-    (property "Reference" "R3" (at 68.58 21.6916 90)
-      (effects (font (size 1.27 1.27)))
-    )
-    (property "Value" "3k" (at 68.58 24.003 90)
-      (effects (font (size 1.27 1.27)))
-    )
-    (property "Footprint" "Resistor_SMD:R_0402_1005Metric" (at 68.58 26.67 0)
-      (effects (font (size 1.27 1.27)) hide)
-    )
-    (property "Datasheet" "~" (at 68.58 26.67 0)
-      (effects (font (size 1.27 1.27)) hide)
-    )
-    (pin "1")
-    (pin "2")
-    (instances
-      (project "RicardoCHEESE"
-        (path "/7db990e4-92e1-4f99-b4d2-435bbec1ba83"
-          (reference "R3") (unit 1)
-        )
-      )
-    )
-  )
   (symbol (lib_id "Connector:TestPoint") (at 29.21 38.1 90) (unit 1)
     (in_bom yes) (on_board yes) (dnp no)
@@
         )
       )
-    )
-  )
-  (symbol (lib_id "power:+12V") (at 73.66 26.67 0) (unit 1)
-    (in_bom yes) (on_board yes) (dnp no)
-    (property "Reference" "#PWR02" (at 73.66 30.48 0)
-      (effects (font (size 1.27 1.27)) hide)
-    )
-    (property "Value" "+12V" (at 73.66 23.114 0)
-      (effects (font (size 1.27 1.27)))
-    )
-    (property "Footprint" "" (at 73.66 26.67 0)
-      (effects (font (size 1.27 1.27)) hide)
-    )
-    (property "Datasheet" "" (at 73.66 26.67 0)
-      (effects (font (size 1.27 1.27)) hide)
-    )
-    (pin "1")
-    (instances
-      (project "RicardoCHEESE"
-        (path "/7db990e4-92e1-4f99-b4d2-435bbec1ba83"
-          (reference "#PWR02") (unit 1)
-        )
-      )

Commit message: ordering
Parts:
- 3V3LED1: value 3V3LED -> BLUE_LED
- TXLED1: value TX_LED -> GREEN_LED
Other:
- note removed: "TBD C and R value to get a total series impedance of 50 ohms at 2.4GHz"
- note removed: "This is the bare minimum required for a board in the Ricardo ecosystem. Please ask before changing or removing anything in this box."
Changed lines of the file:
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@@
-    (effects (font (size 1.27 1.27)) (justify left bottom))
-  )
-  (text "This is the bare minimum required for a board in the Ricardo ecosystem. Please ask before changing or removing anything in this box.\n\n"
-    (at 12.7 13.97 0)
-    (effects (font (size 1.27 1.27)) (justify left bottom))
-  )
-  (text "TBD C and R value to get\na total series impedance\nof 50 ohms at 2.4GHz\n"
-    (at 44.45 55.88 0)
     (effects (font (size 1.27 1.27)) (justify left bottom))
   )
@@
       (effects (font (size 1.27 1.27)))
     )
-    (property "Value" "TX_LED" (at 25.4 24.4856 0)
+    (property "Value" "GREEN_LED" (at 25.4 24.4856 0)
       (effects (font (size 1.27 1.27)))
     )
@@
       (effects (font (size 1.27 1.27)))
     )
-    (property "Value" "3V3LED" (at 54.61 18.6944 0)
-      (effects (font (size 1.27 1.27)))
-    )
+    (property "Value" "BLUE_LED" (at 54.61 18.6944 0)
+      (effects (font (size 1.27 1.27)))
+    )
